Commit message: More Joint State work

File: hexapod_description/urdf/hexapod_model.xacro (robot description, xacro)
@@ -1,123 +1,163 @@
 <?xml version="1.0"?>
-<robot xmlns:xacro="http://ros.org/wiki/xacro" name="hexapod">
-<!-- Build the body frame -->
-    <link name="base_link" />
-    <joint name="base_joint" type="fixed">
-        <parent link="base_link" />
-        <child link="body" />
-        <origin xyz="0 0 0" rpy="0 0 0" />
-    </joint>
-    <link name="body">
-            <visual>
-                <origin xyz="0 0 0" rpy="0 0 0" />
-                <geometry>
-                    <cylinder radius="5" length="5"/>
-                </geometry>
-                <material name="grey">
-                    <color rgba="0.5 0.5 0.5 1" />
-                </material>
-            </visual>
-    </link>
-<!-- Pi parameter -->
-    <xacro:property name="pi" value="3.1415926535897931" />
-<!-- Joint properties -->
-    <xacro:property name="joint_lower_limit" value="-${1.5}" />
-    <xacro:property name="joint_upper_limit" value="${1.5}" />
-    <xacro:property name="joint_effort" value="10000" />
-    <xacro:property name="joint_velocity" value="100" />
-    <!-- Leg macros -->
-    <xacro:macro name="leg" params="side position x y angle">
-<!-- Build leg -->
-        <joint name="${side}${position}_leg_center_joint" type="fixed">
-                <origin xyz="${x} ${y} 0" rpy="0 0 0" />
-                <parent link="body" />
-                <child link="${side}${position}_leg_center" />
-        </joint>
-        <link name="${side}${position}_leg_center" />
-        <joint name="${side}${position}_coxa_joint" type="revolute">
-                <origin xyz="0 0 0" rpy="0 0 ${angle}" />
-                <parent link="${side}${position}_leg_center" />
-                <child link="${side}${position}_coxa" />
-                <axis xyz="0 0 -1" />
-                <limit lower="${joint_lower_limit}" upper="${joint_upper_limit}" effort="${joint_effort}" velocity="${joint_velocity}" />
-        </joint>
-        <link name="${side}${position}_coxa">
-                <visual>
-                    <origin xyz="0 0 0" rpy="0 0 0" />
-                    <geometry>
-                        <cylinder radius="1" length="3"/>
-                    </geometry>
-                    <material name="">
-                        <color rgba="0.7 0.7 0 1" />
-                    </material>
-                </visual>
-        </link>
-        <joint name="${side}${position}_femur_joint" type="revolute">
-                <origin xyz="58.93 0 0" rpy="-${pi/2} 0 0" />
-                <parent link="${side}${position}_coxa" />
-                <child link="${side}${position}_femur" />
-                <axis xyz="0 0 -1" />
-                <limit lower="${joint_lower_limit}" upper="${joint_upper_limit}" effort="${joint_effort}" velocity="${joint_velocity}" />
-        </joint>
-        <link name="${side}${position}_femur">
-                <visual>
-                    <origin xyz="0 0 0" rpy="0 0 0" />
-                    <geometry>
-                        <cylinder radius="1" length="3"/>
-                    </geometry>
-                    <material name="">
-                        <color rgba="0 0.7 0.7 1" />
-                    </material>
-                </visual>
-        </link>
-        <joint name="${side}${position}_tibia_joint" type="revolute">
-                <origin xyz="107.98 0 0" rpy="-${pi/2} 0 0" />
-                <parent link="${side}${position}_femur" />
-                <child link="${side}${position}_tibia" />
-                <axis xyz="0 0 -1" />
-                <limit lower="${joint_lower_limit}" upper="${joint_upper_limit}" effort="${joint_effort}" velocity="${joint_velocity}" />
-        </joint>
-        <link name="${side}${position}_tibia">
-                <visual>
-                    <origin xyz="0 0 0" rpy="0 0 0" />
-                    <geometry>
-                        <cylinder radius="1" length="3"/>
-                    </geometry>
-                    <material name="">
-                        <color rgba="0 0.7 0.7 1" />
-                    </material>
-                </visual>
-        </link>
-        <joint name="${side}${position}_tarsus_joint" type="revolute">
-                <origin xyz="87.74 0 0" rpy="${pi} 0 ${pi/2}" />
-                <parent link="${side}${position}_tibia" />
-                <child link="${side}${position}_tarsus" />
-                <axis xyz="0 0 1" />
-                <limit lower="${joint_lower_limit}" upper="${joint_upper_limit}" effort="${joint_effort}" velocity="${joint_velocity}" />
-        </joint>
-        <link name="${side}${position}_tarsus">
-                <visual>
-                    <origin xyz="0 0 0" rpy="0 0 0" />
-                    <geometry>
-                        <cylinder radius="1" length="3"/>
-                    </geometry>
-                    <material name="">
-                        <color rgba="0.7 0 0.7 1" />
-                    </material>
-                </visual>
-        </link>
-        <joint name="${side}${position}_tarsus_foot_joint" type="fixed">
-                <origin xyz="120.65 0 0" rpy="0 0 0" />
-                <parent link="${side}${position}_tarsus" />
-                <child link="${side}${position}_tarsus_foot" />
-        </joint>
-        <link name="${side}${position}_tarsus_foot" />
-    </xacro:macro>
+<robot xmlns:xacro="http://ros.org/wiki/xacro" name="Golem">
+	<!-- parameters -->
+	<xacro:property name="pi" value="3.1415926535897931" />
+	<xacro:property name="body_length_x" value="0.3556" />
+	<xacro:property name="body_length_y" value="0.165" />
+	<xacro:property name="coxa_length" value="0.05893" />
+	<xacro:property name="femur_length" value="0.10798" />
+	<xacro:property name="tibia_length" value="0.08774" />
+	<xacro:property name="tarsus_length" value="0.12065" />
+	<!-- Build the body frame -->
+	<link name="base_link" />
+	<joint name="base_joint" type="fixed">
+		<parent link="base_link" />
+		<child link="body" />
+		<origin xyz="0 0 0" rpy="0 0 0" />
+	</joint>
+	<link name="body">
+			<visual>
+	  			<origin	xyz="0 0 0" rpy="0 0 0" />
+	  			<geometry>
+					<box size="${body_length_x} ${body_length_y} 0.05"/>
+	  			</geometry>
+	 			<material name="grey">
+					<color rgba="0.5 0.5 0.5 1" />
+	  			</material>
+			</visual>
+	</link>
+	<!-- Joint properties -->
+	<xacro:property name="joint_lower_limit" value="-${1.5}" />
+	<xacro:property name="joint_upper_limit" value="${1.5}" />
+	<xacro:property name="joint_effort" value="10000" />
+	<xacro:property name="joint_velocity" value="100" />
+	<!-- Leg macro -->
+	<xacro:macro name="leg" params="side position x y angle">
+		<!-- leg position -->
+		<joint name="leg_center_joint_${side}${position}" type="fixed">
+			<origin xyz="${x} ${y} 0" rpy="0 0 0" />
+			<parent link="body" />
+			<child link="leg_center_${side}${position}" />
+		</joint>
+		<link name="leg_center_${side}${position}" />
+		<!-- coxa -->
+		<joint name="coxa_joint_${side}${position}" type="revolute">
+			<origin xyz="0 0 0" rpy="0 0 ${angle}" />
+			<parent link="leg_center_${side}${position}" />
+			<child link="coxa_${side}${position}" />
+			<axis xyz="0 0 -1" />
+			<limit lower="${joint_lower_limit}" upper="${joint_upper_limit}" effort="${joint_effort}" velocity="${joint_velocity}" />
+		</joint>
+		<link name="coxa_${side}${position}">
+			<visual>
+				<origin xyz="0 0 0" rpy="0 0 0" />
+				<geometry>
+					<cylinder length="0.0508" radius="0.015875"/>
+				</geometry>
+				<material name="">
+					<color rgba="0.7 0.7 0 1" />
+				</material>
+			</visual>
+			<visual>
+				<origin xyz="${coxa_length/2} 0 0" rpy="0 ${pi/2} 0" />
+				<geometry>
+					<cylinder length="${coxa_length}" radius="0.0127"/>
+				</geometry>
+				<material name="">
+					<color rgba="0.7 0.7 0 1" />
+				</material>
+			</visual>
+		</link>
+		<!-- femur -->
+		<joint name="femur_joint_${side}${position}" type="revolute">
+			<origin xyz="${coxa_length} 0 0" rpy="-${pi/2} 0 0" />
+			<parent link="coxa_${side}${position}" />
+			<child link="femur_${side}${position}" />
+			<axis xyz="0 0 -1" />
+			<limit lower="${joint_lower_limit}" upper="${joint_upper_limit}" effort="${joint_effort}" velocity="${joint_velocity}" />
+		</joint>
+		<link name="femur_${side}${position}">
+			<visual>
+				<origin xyz="0 0 0" rpy="0 0 0" />
+				<geometry>
+					<cylinder length="0.0508" radius="0.015875"/>
+				</geometry>
+				<material name="">
+					<color rgba="0 0.7 0.7 1" />
+				</material>
+			</visual>
+			<visual>
+				<origin xyz="0 -${femur_length/2} 0" rpy="${pi/2} 0 0" />
+				<geometry>
+					<cylinder length="${femur_length}" radius="0.0127"/>
+				</geometry>
+				<material name="">
+					<color rgba="0 0.7 0.7 1" />
+				</material>
+			</visual>
+		</link>
+		<!-- tibia -->
+		<joint name="tibia_joint_${side}${position}" type="revolute">
+			<origin xyz="0 -${femur_length} 0" rpy="${pi} 0 0" />
+			<parent link="femur_${side}${position}" />
+			<child link="tibia_${side}${position}" />
+			<axis xyz="0 0 1" />
+			<limit lower="${joint_lower_limit}" upper="${joint_upper_limit}" effort="${joint_effort}" velocity="${joint_velocity}" />
+		</joint>
+		<link name="tibia_${side}${position}">
+			<visual>
+				<origin xyz="0 0 0" rpy="0 0 0.06" />
+				<geometry>
+					<cylinder length="0.0508" radius="0.015875"/>
+				</geometry>
+				<material name="">
+					<color rgba="0.7 0 0.7 1" />
+				</material>
+			</visual>
+			<visual>
+				<origin xyz="${tibia_length/2} 0 0" rpy="0 ${pi/2} 0" />
+				<geometry>
+					<cylinder length="${tibia_length}" radius="0.0127"/>
+				</geometry>
+				<material name="">
+					<color rgba="0.7 0 0.7 1" />
+				</material>
+			</visual>
+		</link>
+		<!-- tarsus -->
+		<joint name="tarsus_joint_${side}${position}" type="revolute">
+			<origin xyz="${tibia_length} 0 0" rpy="0 0 -${pi/2}" />
+			<parent link="tibia_${side}${position}" />
+			<child link="tarsus_${side}${position}" />
+			<axis xyz="0 0 1" />
+			<limit lower="${joint_lower_limit}" upper="${joint_upper_limit}" effort="${joint_effort}" velocity="${joint_velocity}" />
+		</joint>
+		<link name="tarsus_${side}${position}">
+			<visual>
+				<origin xyz="0 0 0" rpy="0 0 0.06" />
+				<geometry>
+					<cylinder length="0.0508" radius="0.015875"/>
+				</geometry>
+				<material name="">
+					<color rgba="0.7 0.7 0.7 1" />
+				</material>
+			</visual>
+			<visual>
+				<origin xyz="${tarsus_length/2} 0 0" rpy="0 ${pi/2} 0" />
+				<geometry>
+					<cylinder length="${tarsus_length}" radius="0.0127"/>
+				</geometry>
+				<material name="">
+					<color rgba="0.7 0.7 0.7 1" />
+				</material>
+			</visual>
+		</link>
+	</xacro:macro>
 <!-- Build robot model -->
-    <xacro:leg side="R" position="R" x="177.8"  y="-82.5"   angle="-${pi/4}" />
-    <xacro:leg side="R" position="M" x="0.0"    y="-133.35" angle="${pi/2}" />
-    <xacro:leg side="R" position="F" x="-177.8" y="-82.5"   angle="${pi*1/4}" />
-    <xacro:leg side="L" position="R" x="177.8"  y="82.5"    angle="-${pi/4}" />
-    <xacro:leg side="L" position="M" x="0.0"    y="133.35"  angle="${pi/2}" />
-    <xacro:leg side="L" position="F" x="-177.8" y="82.5"    angle="${pi*1/4}" />
+	<xacro:leg side="R" position="R" x="0.1778" y="-0.0825" angle="-${pi/4}" />
+	<xacro:leg side="R" position="M" x="0.0" y="-0.13335" angle="${pi/2}" />
+	<xacro:leg side="R" position="F" x="-0.1778" y="-0.0825" angle="${pi*1/4}" />
+	<xacro:leg side="L" position="R" x="0.1778" y="0.0825" angle="-${pi/4}" />
+	<xacro:leg side="L" position="M" x="0.0" y="0.13335" angle="${pi/2}" />
+	<xacro:leg side="L" position="F" x="-0.1778" y="0.0825" angle="${pi*1/4}" />
 </robot>

Commit message: Robot state publisher up and running.

File: hexapod_description/urdf/hexapod_model.xacro (robot description, xacro)
@@ -23,15 +23,15 @@
 	  			</geometry>
 	 			<material name="grey">
-					<color rgba="0.5 0.5 0.5 1" />
+					<color rgba="0.7 0.7 0.7 1" />
 	  			</material>
 			</visual>
 	</link>
 	<!-- Joint properties -->
-	<xacro:property name="joint_lower_limit" value="-${1.5}" />
-	<xacro:property name="joint_upper_limit" value="${1.5}" />
+	<xacro:property name="joint_lower_limit" value="-${3.14}" />
+	<xacro:property name="joint_upper_limit" value="${3.14}" />
 	<xacro:property name="joint_effort" value="10000" />
 	<xacro:property name="joint_velocity" value="100" />
 	<!-- Leg macro -->
-	<xacro:macro name="leg" params="side position x y angle">
+	<xacro:macro name="leg" params="side position x y angle axis">
 		<!-- leg position -->
 		<joint name="leg_center_joint_${side}${position}" type="fixed">
@@ -46,5 +46,5 @@
 			<parent link="leg_center_${side}${position}" />
 			<child link="coxa_${side}${position}" />
-			<axis xyz="0 0 -1" />
+			<axis xyz="0 0 ${axis}" />
 			<limit lower="${joint_lower_limit}" upper="${joint_upper_limit}" effort="${joint_effort}" velocity="${joint_velocity}" />
 		</joint>
@@ -56,5 +56,5 @@
 				</geometry>
 				<material name="">
-					<color rgba="0.7 0.7 0 1" />
+					<color rgba="0.7 0.7 0.7 1" />
 				</material>
 			</visual>
@@ -65,5 +65,5 @@
 				</geometry>
 				<material name="">
-					<color rgba="0.7 0.7 0 1" />
+					<color rgba="0.7 0.7 0.7 1" />
 				</material>
 			</visual>
@@ -74,5 +74,5 @@
 			<parent link="coxa_${side}${position}" />
 			<child link="femur_${side}${position}" />
-			<axis xyz="0 0 -1" />
+			<axis xyz="0 0 ${axis*-1}" />
 			<limit lower="${joint_lower_limit}" upper="${joint_upper_limit}" effort="${joint_effort}" velocity="${joint_velocity}" />
 		</joint>
@@ -84,5 +84,5 @@
 				</geometry>
 				<material name="">
-					<color rgba="0 0.7 0.7 1" />
+					<color rgba="0.7 0.7 0.7 1" />
 				</material>
 			</visual>
@@ -93,5 +93,5 @@
 				</geometry>
 				<material name="">
-					<color rgba="0 0.7 0.7 1" />
+					<color rgba="0.7 0.7 0.7 1" />
 				</material>
 			</visual>
@@ -102,5 +102,5 @@
 			<parent link="femur_${side}${position}" />
 			<child link="tibia_${side}${position}" />
-			<axis xyz="0 0 1" />
+			<axis xyz="0 0 ${axis*-1}" />
 			<limit lower="${joint_lower_limit}" upper="${joint_upper_limit}" effort="${joint_effort}" velocity="${joint_velocity}" />
 		</joint>
@@ -112,5 +112,5 @@
 				</geometry>
 				<material name="">
-					<color rgba="0.7 0 0.7 1" />
+					<color rgba="0.7 0.7 0.7 1" />
 				</material>
 			</visual>
@@ -121,5 +121,5 @@
 				</geometry>
 				<material name="">
-					<color rgba="0.7 0 0.7 1" />
+					<color rgba="0.7 0.7 0.7 1" />
 				</material>
 			</visual>
@@ -130,5 +130,5 @@
 			<parent link="tibia_${side}${position}" />
 			<child link="tarsus_${side}${position}" />
-			<axis xyz="0 0 1" />
+			<axis xyz="0 0 ${axis*-1}" />
 			<limit lower="${joint_lower_limit}" upper="${joint_upper_limit}" effort="${joint_effort}" velocity="${joint_velocity}" />
 		</joint>
@@ -155,9 +155,9 @@
 	</xacro:macro>
 <!-- Build robot model -->
-	<xacro:leg side="R" position="R" x="0.1778" y="-0.0825" angle="-${pi/4}" />
-	<xacro:leg side="R" position="M" x="0.0" y="-0.13335" angle="${pi/2}" />
-	<xacro:leg side="R" position="F" x="-0.1778" y="-0.0825" angle="${pi*1/4}" />
-	<xacro:leg side="L" position="R" x="0.1778" y="0.0825" angle="-${pi/4}" />
-	<xacro:leg side="L" position="M" x="0.0" y="0.13335" angle="${pi/2}" />
-	<xacro:leg side="L" position="F" x="-0.1778" y="0.0825" angle="${pi*1/4}" />
+	<xacro:leg side="R" position="R" x="0.1778" y="-0.0825" angle="-${pi/4}" axis="-1" />
+	<xacro:leg side="R" position="M" x="0.0" y="-0.13335" angle="-${pi/2}" axis="-1" />
+	<xacro:leg side="R" position="F" x="-0.1778" y="-0.0825" angle="-${pi*3/4}" axis="-1" />
+	<xacro:leg side="L" position="R" x="0.1778" y="0.0825" angle="${pi/4}" axis="1" />
+	<xacro:leg side="L" position="M" x="0.0" y="0.13335" angle="${pi/2}" axis="1" />
+	<xacro:leg side="L" position="F" x="-0.1778" y="0.0825" angle="${pi*3/4}" axis="1" />
 </robot>

Commit message: Added models for body, coxa and femur

File: hexapod_description/urdf/hexapod_model.xacro (robot description, xacro)
@@ -19,10 +19,10 @@
 			<visual>
 	  			<origin	xyz="0 0 0" rpy="0 0 0" />
-	  			<geometry>
-					<box size="${body_length_x} ${body_length_y} 0.05"/>
-	  			</geometry>
-	 			<material name="grey">
+      			<geometry>
+        			<mesh filename="package://hexapod_description/meshes/body.stl" />
+      			</geometry>
+				<material name="">
 					<color rgba="0.7 0.7 0.7 1" />
-	  			</material>
+				</material>
 			</visual>
 	</link>
@@ -52,16 +52,7 @@
 			<visual>
 				<origin xyz="0 0 0" rpy="0 0 0" />
-				<geometry>
-					<cylinder length="0.0508" radius="0.015875"/>
-				</geometry>
-				<material name="">
-					<color rgba="0.7 0.7 0.7 1" />
-				</material>
-			</visual>
-			<visual>
-				<origin xyz="${coxa_length/2} 0 0" rpy="0 ${pi/2} 0" />
-				<geometry>
-					<cylinder length="${coxa_length}" radius="0.0127"/>
-				</geometry>
+      			<geometry>
+        			<mesh filename="package://hexapod_description/meshes/coxa.stl" />
+      			</geometry>
 				<material name="">
 					<color rgba="0.7 0.7 0.7 1" />
@@ -80,16 +71,7 @@
 			<visual>
 				<origin xyz="0 0 0" rpy="0 0 0" />
-				<geometry>
-					<cylinder length="0.0508" radius="0.015875"/>
-				</geometry>
-				<material name="">
-					<color rgba="0.7 0.7 0.7 1" />
-				</material>
-			</visual>
-			<visual>
-				<origin xyz="0 -${femur_length/2} 0" rpy="${pi/2} 0 0" />
-				<geometry>
-					<cylinder length="${femur_length}" radius="0.0127"/>
-				</geometry>
+      			<geometry>
+        			<mesh filename="package://hexapod_description/meshes/femur.stl" />
+      			</geometry>
 				<material name="">
 					<color rgba="0.7 0.7 0.7 1" />

Commit message: rviz model tweaks

File: hexapod_description/urdf/hexapod_model.xacro (robot description, xacro)
@@ -20,5 +20,5 @@
 	  			<origin	xyz="0 0 0" rpy="0 0 0" />
       			<geometry>
-        			<mesh filename="package://hexapod_description/meshes/body.stl" />
+        			<mesh filename="package://hexapod_description/meshes/body.stl" scale="0.001 0.001 0.001"/>
       			</geometry>
 				<material name="">
@@ -53,5 +53,5 @@
 				<origin xyz="0 0 0" rpy="0 0 0" />
       			<geometry>
-        			<mesh filename="package://hexapod_description/meshes/coxa.stl" />
+        			<mesh filename="package://hexapod_description/meshes/coxa.stl" scale="0.001 0.001 0.001"/>
       			</geometry>
 				<material name="">
@@ -65,5 +65,5 @@
 			<parent link="coxa_${side}${position}" />
 			<child link="femur_${side}${position}" />
-			<axis xyz="0 0 ${axis*-1}" />
+			<axis xyz="0 0 ${axis}" />
 			<limit lower="${joint_lower_limit}" upper="${joint_upper_limit}" effort="${joint_effort}" velocity="${joint_velocity}" />
 		</joint>
@@ -72,5 +72,5 @@
 				<origin xyz="0 0 0" rpy="0 0 0" />
       			<geometry>
-        			<mesh filename="package://hexapod_description/meshes/femur.stl" />
+        			<mesh filename="package://hexapod_description/meshes/femur.stl" scale="0.001 0.001 0.001"/>
       			</geometry>
 				<material name="">
@@ -84,22 +84,13 @@
 			<parent link="femur_${side}${position}" />
 			<child link="tibia_${side}${position}" />
-			<axis xyz="0 0 ${axis*-1}" />
+			<axis xyz="0 0 ${axis}" />
 			<limit lower="${joint_lower_limit}" upper="${joint_upper_limit}" effort="${joint_effort}" velocity="${joint_velocity}" />
 		</joint>
 		<link name="tibia_${side}${position}">
 			<visual>
-				<origin xyz="0 0 0" rpy="0 0 0.06" />
-				<geometry>
-					<cylinder length="0.0508" radius="0.015875"/>
-				</geometry>
-				<material name="">
-					<color rgba="0.7 0.7 0.7 1" />
-				</material>
-			</visual>
-			<visual>
-				<origin xyz="${tibia_length/2} 0 0" rpy="0 ${pi/2} 0" />
-				<geometry>
-					<cylinder length="${tibia_length}" radius="0.0127"/>
-				</geometry>
+				<origin xyz="0 0 0" rpy="0 0 0" />
+      			<geometry>
+        			<mesh filename="package://hexapod_description/meshes/tibia.stl" scale="0.001 0.001 0.001"/>
+      			</geometry>
 				<material name="">
 					<color rgba="0.7 0.7 0.7 1" />
@@ -112,22 +103,13 @@
 			<parent link="tibia_${side}${position}" />
 			<child link="tarsus_${side}${position}" />
-			<axis xyz="0 0 ${axis*-1}" />
+			<axis xyz="0 0 ${axis}" />
 			<limit lower="${joint_lower_limit}" upper="${joint_upper_limit}" effort="${joint_effort}" velocity="${joint_velocity}" />
 		</joint>
 		<link name="tarsus_${side}${position}">
 			<visual>
-				<origin xyz="0 0 0" rpy="0 0 0.06" />
-				<geometry>
-					<cylinder length="0.0508" radius="0.015875"/>
-				</geometry>
-				<material name="">
-					<color rgba="0.7 0.7 0.7 1" />
-				</material>
-			</visual>
-			<visual>
-				<origin xyz="${tarsus_length/2} 0 0" rpy="0 ${pi/2} 0" />
-				<geometry>
-					<cylinder length="${tarsus_length}" radius="0.0127"/>
-				</geometry>
+				<origin xyz="0 0 0" rpy="0 0 0" />
+      			<geometry>
+        			<mesh filename="package://hexapod_description/meshes/tarsus.stl" scale="0.001 0.001 0.001"/>
+      			</geometry>
 				<material name="">
 					<color rgba="0.7 0.7 0.7 1" />
@@ -137,9 +119,9 @@
 	</xacro:macro>
 <!-- Build robot model -->
-	<xacro:leg side="R" position="R" x="0.1778" y="-0.0825" angle="-${pi/4}" axis="-1" />
-	<xacro:leg side="R" position="M" x="0.0" y="-0.13335" angle="-${pi/2}" axis="-1" />
-	<xacro:leg side="R" position="F" x="-0.1778" y="-0.0825" angle="-${pi*3/4}" axis="-1" />
-	<xacro:leg side="L" position="R" x="0.1778" y="0.0825" angle="${pi/4}" axis="1" />
-	<xacro:leg side="L" position="M" x="0.0" y="0.13335" angle="${pi/2}" axis="1" />
-	<xacro:leg side="L" position="F" x="-0.1778" y="0.0825" angle="${pi*3/4}" axis="1" />
+	<xacro:leg side="R" position="R" x="0.1778" y="-0.0825" angle="-${pi/4}" axis="1" />
+	<xacro:leg side="R" position="M" x="0.0" y="-0.13335" angle="-${pi/2}" axis="1" />
+	<xacro:leg side="R" position="F" x="-0.1778" y="-0.0825" angle="-${pi*3/4}" axis="1" />
+	<xacro:leg side="L" position="R" x="0.1778" y="0.0825" angle="${pi/4}" axis="-1" />
+	<xacro:leg side="L" position="M" x="0.0" y="0.13335" angle="${pi/2}" axis="-1" />
+	<xacro:leg side="L" position="F" x="-0.1778" y="0.0825" angle="${pi*3/4}" axis="-1" />
 </robot>

Commit message: publish before major change

File: hexapod_description/urdf/hexapod_model.xacro (robot description, xacro)
@@ -10,4 +10,10 @@
 	<xacro:property name="tarsus_length" value="0.12065" />
 	<!-- Build the body frame -->
+    <link name="footprint" />
+    <joint name="footprint_joint" type="fixed">
+        <parent link="footprint"/>
+        <child link="base_link"/>
+		<origin xyz="0 0 0" rpy="0 0 0" />
+    </joint>
 	<link name="base_link" />
 	<joint name="base_joint" type="fixed">
