Commit message: Syncing with Romain Reignier fork of gazebo work

File: hexapod_description/urdf/hexapod_model.xacro (robot description, xacro)
@@ -9,131 +9,334 @@
     <xacro:property name="tibia_length" value="0.08774"/>
     <xacro:property name="tarsus_length" value="0.12065"/>
+    <gazebo>
+        <plugin name="gazebo_ros_control" filename="libgazebo_ros_control.so">
+            <robotNamespace>/Golem</robotNamespace>
+        </plugin>
+    </gazebo>
     <link name="base_link"/>
     <joint name="base_joint" type="fixed">
-      <parent link="base_link"/>
-      <child link="body_link"/>
-      <origin xyz="0.0 0.0 0.0" rpy="0.0 0.0 0.0"/>
+        <parent link="base_link"/>
+        <child link="body_link"/>
+        <origin xyz="0.0 0.0 0.0" rpy="0.0 0.0 0.0"/>
     </joint>
     <link name="body_link">
         <visual>
-          <origin xyz="0.0 0.0 0.0" rpy="0.0 0.0 0.0"/>
-          <geometry>
-            <mesh filename="package://hexapod_description/meshes/body.stl" scale="0.001 0.001 0.001"/>
-          </geometry>
-          <material name="">
-            <color rgba="0.7 0.7 0.7 1"/>
-          </material>
+            <origin xyz="0.0 0.0 0.0" rpy="0.0 0.0 0.0"/>
+            <geometry>
+                <mesh filename="package://hexapod_description/meshes/body.stl" scale="0.001 0.001 0.001"/>
+            </geometry>
+            <material name="">
+                <color rgba="0.7 0.7 0.7 1"/>
+            </material>
         </visual>
+        <collision>
+            <origin xyz="0.0 0.0 0.0" rpy="0.0 0.0 0.0"/>
+            <geometry>
+                <mesh filename="package://hexapod_description/meshes/body.stl" scale="0.001 0.001 0.001"/>
+            </geometry>
+            <material name="">
+                <color rgba="0.7 0.7 0.7 1"/>
+            </material>
+        </collision>
+        <inertial>
+            <origin xyz="0.0 0.0 0.0" rpy="0.0 0.0 0.0" />
+            <mass value="0.00001"/>
+            <inertia
+                ixx="1.0" ixy="0.0"  ixz="0.0"
+                iyy="1.0" iyz="0.0"
+                izz="1.0" />
+        </inertial>
     </link>
+    <gazebo reference="body_link">
+        <material>Gazebo/DarkGrey</material>
+    </gazebo>
     <!-- Camera properties -->
     <joint name="camera_rgb_joint" type="fixed">
-      <parent link="body_link"/>
-      <child link="camera_rgb_optical_frame"/>
-      <origin xyz="0.150 0.0255 0.034" rpy="${pi/2} ${pi} ${pi/2}"/>
+        <parent link="body_link"/>
+        <child link="camera_rgb_optical_frame"/>
+        <origin xyz="0.150 0.0255 0.034" rpy="${pi/2} ${pi} ${pi/2}"/>
     </joint>
-    <link name="camera_rgb_optical_frame"/>
+    <link name="camera_rgb_optical_frame">
+        <inertial>
+            <origin xyz="0.0 0.0 0.0" rpy="0.0 0.0 0.0" />
+            <mass value="0.00001"/>
+            <inertia
+                ixx="1.0" ixy="0.0"  ixz="0.0"
+                iyy="1.0" iyz="0.0"
+                izz="1.0" />
+        </inertial>
+	</link>
     <joint name="camera_depth_joint" type="fixed">
-      <parent link="body_link"/>
-      <child link="camera_depth_optical_frame"/>
-      <origin xyz="0.150 -0.0225 0.034" rpy="${pi/2} ${pi} ${pi/2}"/>
+        <parent link="body_link"/>
+        <child link="camera_depth_optical_frame"/>
+        <origin xyz="0.150 -0.0225 0.034" rpy="${pi/2} ${pi} ${pi/2}"/>
     </joint>
-    <link name="camera_depth_optical_frame"/>
+    <link name="camera_depth_optical_frame">
+        <inertial>
+            <origin xyz="0.0 0.0 0.0" rpy="0.0 0.0 0.0" />
+            <mass value="0.00001"/>
+            <inertia
+                ixx="1.0" ixy="0.0"  ixz="0.0"
+                iyy="1.0" iyz="0.0"
+                izz="1.0" />
+        </inertial>
+	</link>
     <!-- IMU properties -->
     <joint name="imu_joint" type="fixed">
-      <parent link="base_link"/>
-      <child link="imu_link"/>
-      <origin xyz="0.0 0.0 0.034" rpy="${pi} 0.0 0.0"/>
+        <parent link="base_link"/>
+        <child link="imu_link"/>
+        <origin xyz="0.0 0.0 0.034" rpy="${pi} 0.0 0.0"/>
     </joint>
-    <link name="imu_link"/>
+    <link name="imu_link">
+        <inertial>
+            <origin xyz="0.0 0.0 0.0" rpy="0.0 0.0 0.0" />
+            <mass value="0.00001"/>
+            <inertia
+                ixx="1.0" ixy="0.0"  ixz="0.0"
+                iyy="1.0" iyz="0.0"
+                izz="1.0" />
+        </inertial>
+	</link>
     <!-- Joint properties -->
     <xacro:property name="joint_lower_limit" value="-${3.14}"/>
     <xacro:property name="joint_upper_limit" value="${3.14}"/>
-    <xacro:property name="joint_effort" value="10000"/>
-    <xacro:property name="joint_velocity" value="100"/>
+    <xacro:property name="joint_effort" value="6.0"/>
+    <xacro:property name="joint_velocity" value="0.524"/>
     <!-- Leg macro -->
     <xacro:macro name="leg" params="side position x y angle axis">
         <!-- leg position -->
         <joint name="leg_center_joint_${side}${position}" type="fixed">
-          <origin xyz="${x} ${y} 0.0" rpy="0.0 0.0 0.0"/>
-          <parent link="body_link"/>
-          <child link="leg_center_${side}${position}"/>
-        </joint>
-        <link name="leg_center_${side}${position}"/>
+            <origin xyz="${x} ${y} 0.0" rpy="0.0 0.0 0.0"/>
+            <parent link="body_link"/>
+            <child link="leg_center_${side}${position}"/>
+        </joint>
+        <link name="leg_center_${side}${position}">
+			<inertial>
+				<origin xyz="0.0 0.0 0.0" rpy="0.0 0.0 0.0" />
+				<mass value="0.00001"/>
+				<inertia
+					ixx="1.0" ixy="0.0"  ixz="0.0"
+					iyy="1.0" iyz="0.0"
+					izz="1.0" />
+			</inertial>
+		</link>
         <!-- coxa -->
         <joint name="coxa_joint_${side}${position}" type="revolute">
-          <origin xyz="0.0 0.0 0.0" rpy="0.0 0.0 ${angle}"/>
-          <parent link="leg_center_${side}${position}"/>
-          <child link="coxa_${side}${position}"/>
-          <axis xyz="0.0 0.0 ${-axis}"/>
-          <limit lower="${joint_lower_limit}" upper="${joint_upper_limit}" effort="${joint_effort}" velocity="${joint_velocity}"/>
-        </joint>
+            <origin xyz="0.0 0.0 0.0" rpy="0.0 0.0 ${angle}"/>
+            <parent link="leg_center_${side}${position}"/>
+            <child link="coxa_${side}${position}"/>
+            <axis xyz="0.0 0.0 ${-axis}"/>
+            <limit lower="${joint_lower_limit}" upper="${joint_upper_limit}" effort="${joint_effort}" velocity="${joint_velocity}"/>
+        </joint>
+        <transmission name="coxa_transmission_${side}${position}">
+            <type>transmission_interface/SimpleTransmission</type>
+            <joint name="coxa_joint_${side}${position}">
+                <hardwareInterface>EffortJointInterface</hardwareInterface>
+            </joint>
+            <actuator name="coxa_motor_${side}${position}">
+                <hardwareInterface>EffortJointInterface</hardwareInterface>
+                <mechanicalReduction>1</mechanicalReduction>
+            </actuator>
+        </transmission>
         <link name="coxa_${side}${position}">
-          <visual>
-            <origin xyz="0.0 0.0 0.0" rpy="0.0 0.0 0.0"/>
-            <geometry>
-              <mesh filename="package://hexapod_description/meshes/coxa.stl" scale="0.001 0.001 0.001"/>
-            </geometry>
-            <material name="">
-              <color rgba="0.7 0.7 0.7 1"/>
-            </material>
-          </visual>
+            <visual>
+                <origin xyz="0.0 0.0 0.0" rpy="0.0 0.0 0.0"/>
+                <geometry>
+                    <mesh filename="package://hexapod_description/meshes/coxa.stl" scale="0.001 0.001 0.001"/>
+                </geometry>
+                <material name="">
+                    <color rgba="0.7 0.7 0.7 1"/>
+                </material>
+            </visual>
+            <collision>
+                <origin xyz="0.0 0.0 0.0" rpy="0.0 0.0 0.0" />
+                <geometry>
+                    <mesh filename="package://hexapod_description/meshes/coxa.stl" scale="0.001 0.001 0.001"/>
+                </geometry>
+                <material name="">
+                    <color rgba="0.7 0.7 0.7 1" />
+                </material>
+            </collision>
+            <inertial>
+                <origin xyz="0.0 0.0 0.0" rpy="0.0 0.0 0.0" />
+                <mass value="0.00001"/>
+                <inertia
+                    ixx="1.0" ixy="0.0"  ixz="0.0"
+                    iyy="1.0" iyz="0.0"
+                    izz="1.0" />
+            </inertial>
         </link>
+        <gazebo reference="coxa_${side}${position}">
+            <material>Gazebo/DarkGrey</material>
+        </gazebo>
         <!-- femur -->
         <joint name="femur_joint_${side}${position}" type="revolute">
-          <origin xyz="${coxa_length} 0.0 0.0" rpy="-${pi/2} 0.0 0.0"/>
-          <parent link="coxa_${side}${position}"/>
-          <child link="femur_${side}${position}"/>
-          <axis xyz="0.0 0.0 ${axis}"/>
-          <limit lower="${joint_lower_limit}" upper="${joint_upper_limit}" effort="${joint_effort}" velocity="${joint_velocity}"/>
-        </joint>
+            <origin xyz="${coxa_length} 0.0 0.0" rpy="-${pi/2} 0.0 0.0"/>
+            <parent link="coxa_${side}${position}"/>
+            <child link="femur_${side}${position}"/>
+            <axis xyz="0.0 0.0 ${axis}"/>
+            <limit lower="${joint_lower_limit}" upper="${joint_upper_limit}" effort="${joint_effort}" velocity="${joint_velocity}"/>
+        </joint>
+        <transmission name="femur_transmission_${side}${position}">
+            <type>transmission_interface/SimpleTransmission</type>
+            <joint name="femur_joint_${side}${position}">
+                <hardwareInterface>EffortJointInterface</hardwareInterface>
+            </joint>
+            <actuator name="femur_motor_${side}${position}">
+                <hardwareInterface>EffortJointInterface</hardwareInterface>
+                <mechanicalReduction>1</mechanicalReduction>
+            </actuator>
+        </transmission>
         <link name="femur_${side}${position}">
-          <visual>
-            <origin xyz="0.0 0.0 0.0" rpy="0.0 0.0 0.0"/>
-            <geometry>
-              <mesh filename="package://hexapod_description/meshes/femur.stl" scale="0.001 0.001 0.001"/>
-            </geometry>
-            <material name="">
-              <color rgba="0.7 0.7 0.7 1"/>
-            </material>
-          </visual>
+            <visual>
+                <origin xyz="0.0 0.0 0.0" rpy="0.0 0.0 0.0"/>
+                <geometry>
+                    <mesh filename="package://hexapod_description/meshes/femur.stl" scale="0.001 0.001 0.001"/>
+                </geometry>
+                <material name="">
+                    <color rgba="0.7 0.7 0.7 1"/>
+                </material>
+            </visual>
+            <collision>
+                <origin xyz="0.0 0.0 0.0" rpy="0.0 0.0 0.0" />
+                <geometry>
+                    <mesh filename="package://hexapod_description/meshes/femur.stl" scale="0.001 0.001 0.001"/>
+                </geometry>
+                <material name="">
+                    <color rgba="0.7 0.7 0.7 1" />
+                </material>
+            </collision>
+            <inertial>
+                <origin xyz="0.0 0.0 0.0" rpy="0.0 0.0 0.0" />
+                <mass value="0.00001"/>
+                <inertia
+                    ixx="1.0" ixy="0.0"  ixz="0.0"
+                    iyy="1.0" iyz="0.0"
+                    izz="1.0" />
+            </inertial>
         </link>
         <!-- tibia -->
         <joint name="tibia_joint_${side}${position}" type="revolute">
-          <origin xyz="0.0 -${femur_length} 0.0" rpy="${pi} 0.0 0.0"/>
-          <parent link="femur_${side}${position}"/>
-          <child link="tibia_${side}${position}"/>
-          <axis xyz="0.0 0.0 ${axis}"/>
-          <limit lower="${joint_lower_limit}" upper="${joint_upper_limit}" effort="${joint_effort}" velocity="${joint_velocity}"/>
-        </joint>
+            <origin xyz="0.0 -${femur_length} 0.0" rpy="${pi} 0.0 0.0"/>
+            <parent link="femur_${side}${position}"/>
+            <child link="tibia_${side}${position}"/>
+            <axis xyz="0.0 0.0 ${axis}"/>
+            <limit lower="${joint_lower_limit}" upper="${joint_upper_limit}" effort="${joint_effort}" velocity="${joint_velocity}"/>
+        </joint>
+        <transmission name="tibia_transmission_${side}${position}">
+            <type>transmission_interface/SimpleTransmission</type>
+            <joint name="tibia_joint_${side}${position}">
+                <hardwareInterface>EffortJointInterface</hardwareInterface>
+            </joint>
+            <actuator name="tibia_motor_${side}${position}">
+                <hardwareInterface>EffortJointInterface</hardwareInterface>
+                <mechanicalReduction>1</mechanicalReduction>
+            </actuator>
+        </transmission>
         <link name="tibia_${side}${position}">
-          <visual>
-            <origin xyz="0.0 0.0 0.0" rpy="0.0 0.0 0.0"/>
-            <geometry>
-              <mesh filename="package://hexapod_description/meshes/tibia.stl" scale="0.001 0.001 0.001"/>
-            </geometry>
-            <material name="">
-              <color rgba="0.7 0.7 0.7 1"/>
-            </material>
-          </visual>
+            <visual>
+                <origin xyz="0.0 0.0 0.0" rpy="0.0 0.0 0.0"/>
+                <geometry>
+                    <mesh filename="package://hexapod_description/meshes/tibia.stl" scale="0.001 0.001 0.001"/>
+                </geometry>
+                <material name="">
+                    <color rgba="0.7 0.7 0.7 1"/>
+                </material>
+            </visual>
+            <collision>
+                <origin xyz="0.0 0.0 0.0" rpy="0.0 0.0 0.0" />
+                <geometry>
+                    <mesh filename="package://hexapod_description/meshes/tibia.stl" scale="0.001 0.001 0.001"/>
+                </geometry>
+                <material name="">
+                    <color rgba="0.7 0.7 0.7 1" />
+                </material>
+            </collision>
+            <inertial>
+                <origin xyz="0.0 0.0 0.0" rpy="0.0 0.0 0.0" />
+                <mass value="0.00001"/>
+                <inertia
+                    ixx="1.0" ixy="0.0"  ixz="0.0"
+                    iyy="1.0" iyz="0.0"
+                    izz="1.0" />
+            </inertial>
         </link>
+        <gazebo reference="tibia_${side}${position}">
+            <material>Gazebo/DarkGrey</material>
+        </gazebo>
         <!-- tarsus -->
         <joint name="tarsus_joint_${side}${position}" type="revolute">
-          <origin xyz="${tibia_length} 0.0 0.0" rpy="0.0 0.0 -${pi/2}"/>
-          <parent link="tibia_${side}${position}"/>
-          <child link="tarsus_${side}${position}"/>
-          <axis xyz="0.0 0.0 ${axis}"/>
-          <limit lower="${joint_lower_limit}" upper="${joint_upper_limit}" effort="${joint_effort}" velocity="${joint_velocity}"/>
-        </joint>
+            <origin xyz="${tibia_length} 0.0 0.0" rpy="0.0 0.0 -${pi/2}"/>
+            <parent link="tibia_${side}${position}"/>
+            <child link="tarsus_${side}${position}"/>
+            <axis xyz="0.0 0.0 ${axis}"/>
+            <limit lower="${joint_lower_limit}" upper="${joint_upper_limit}" effort="${joint_effort}" velocity="${joint_velocity}"/>
+        </joint>
+        <transmission name="tarsus_transmission_${side}${position}">
+            <type>transmission_interface/SimpleTransmission</type>
+            <joint name="tarsus_joint_${side}${position}">
+                <hardwareInterface>EffortJointInterface</hardwareInterface>
+            </joint>
+            <actuator name="tarsus_motor_${side}${position}">
+                <hardwareInterface>EffortJointInterface</hardwareInterface>
+                <mechanicalReduction>1</mechanicalReduction>
+            </actuator>
+        </transmission>
         <link name="tarsus_${side}${position}">
-          <visual>
-            <origin xyz="0.0 0.0 0.0" rpy="0.0 0.0 0.0"/>
-            <geometry>
-              <mesh filename="package://hexapod_description/meshes/tarsus.stl" scale="0.001 0.001 0.001"/>
-            </geometry>
-            <material name="">
-              <color rgba="0.7 0.7 0.7 1"/>
-            </material>
-          </visual>
+            <visual>
+                <origin xyz="0.0 0.0 0.0" rpy="0.0 0.0 0.0"/>
+                <geometry>
+                    <mesh filename="package://hexapod_description/meshes/tarsus.stl" scale="0.001 0.001 0.001"/>
+                </geometry>
+                <material name="">
+                    <color rgba="0.7 0.7 0.7 1"/>
+                </material>
+            </visual>
+            <collision>
+                <origin xyz="0.0 0.0 0.0" rpy="0.0 0.0 0.0" />
+                <geometry>
+                    <mesh filename="package://hexapod_description/meshes/tarsus.stl" scale="0.001 0.001 0.001"/>
+                </geometry>
+                <material name="">
+                    <color rgba="0.7 0.7 0.7 1" />
+                </material>
+            </collision>
+            <inertial>
+                <origin xyz="0.0 0.0 0.0" rpy="0.0 0.0 0.0" />
+                <mass value="0.00001"/>
+                <inertia
+                    ixx="1.0" ixy="0.0"  ixz="0.0"
+                    iyy="1.0" iyz="0.0"
+                    izz="1.0" />
+            </inertial>
         </link>
+        <gazebo reference="tarsus_${side}${position}">
+            <material>Gazebo/DarkGrey</material>
+        </gazebo>
+        <!-- foot -->
+        <joint name="foot_joint_${side}${position}" type="fixed">
+            <origin xyz="${tarsus_length} 0.0 0.0" rpy="0.0 0.0 0.0" />
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
Commit message: Joint State publisher and URDF fixes.

File: hexapod_description/urdf/hexapod_model.xacro (robot description, xacro)
@@ -126,5 +126,5 @@
             <parent link="leg_center_${side}${position}"/>
             <child link="coxa_${side}${position}"/>
-            <axis xyz="0.0 0.0 ${-axis}"/>
+            <axis xyz="0.0 0.0 1.0"/>
             <limit lower="${joint_lower_limit}" upper="${joint_upper_limit}" effort="${joint_effort}" velocity="${joint_velocity}"/>
         </joint>
@@ -172,5 +172,5 @@
         <!-- femur -->
         <joint name="femur_joint_${side}${position}" type="revolute">
-            <origin xyz="${coxa_length} 0.0 0.0" rpy="-${pi/2} 0.0 0.0"/>
+            <origin xyz="${coxa_length} 0.0 0.0" rpy="-${pi/2} ${pi/2} 0.0"/>
             <parent link="coxa_${side}${position}"/>
             <child link="femur_${side}${position}"/>
@@ -267,5 +267,5 @@
         <!-- tarsus -->
         <joint name="tarsus_joint_${side}${position}" type="revolute">
-            <origin xyz="${tibia_length} 0.0 0.0" rpy="0.0 0.0 -${pi/2}"/>
+            <origin xyz="${tibia_length} 0.0 0.0" rpy="0.0 0.0 0.0"/>
             <parent link="tibia_${side}${position}"/>
             <child link="tarsus_${side}${position}"/>

Commit message: Base msg change and jointState improvements

File: hexapod_description/urdf/hexapod_model.xacro (robot description, xacro)
@@ -103,4 +103,22 @@
     <xacro:property name="joint_effort" value="6.0"/>
     <xacro:property name="joint_velocity" value="0.524"/>
+    <!-- Head properties -->
+    <joint name="pan_joint" type="revolute">
+        <parent link="body_link"/>
+        <child link="pan_link"/>
+        <origin xyz="0.1 0.0 0.034" rpy="0.0 0.0 0.0"/>
+		<axis xyz="0.0 0.0 1.0"/>
+		<limit lower="${joint_lower_limit}" upper="${joint_upper_limit}" effort="${joint_effort}" velocity="${joint_velocity}"/>
+    </joint>
+    <link name="pan_link">
+        <inertial>
+            <origin xyz="0.0 0.0 0.0" rpy="0.0 0.0 0.0" />
+            <mass value="0.00001"/>
+            <inertia
+                ixx="1.0" ixy="0.0"  ixz="0.0"
+                iyy="1.0" iyz="0.0"
+                izz="1.0" />
+        </inertial>
+	</link>
     <!-- Leg macro -->
     <xacro:macro name="leg" params="side position x y angle axis">

Commit message: Tab/Space cleanup

File: hexapod_description/urdf/hexapod_model.xacro (robot description, xacro)
@@ -66,5 +66,5 @@
                 izz="1.0" />
         </inertial>
-	</link>
+    </link>
     <joint name="camera_depth_joint" type="fixed">
         <parent link="body_link"/>
@@ -81,5 +81,5 @@
                 izz="1.0" />
         </inertial>
-	</link>
+    </link>
     <!-- IMU properties -->
     <joint name="imu_joint" type="fixed">
@@ -97,5 +97,5 @@
                 izz="1.0" />
         </inertial>
-	</link>
+    </link>
     <!-- Joint properties -->
     <xacro:property name="joint_lower_limit" value="-${3.14}"/>
@@ -108,6 +108,6 @@
         <child link="pan_link"/>
         <origin xyz="0.1 0.0 0.034" rpy="0.0 0.0 0.0"/>
-		<axis xyz="0.0 0.0 1.0"/>
-		<limit lower="${joint_lower_limit}" upper="${joint_upper_limit}" effort="${joint_effort}" velocity="${joint_velocity}"/>
+        <axis xyz="0.0 0.0 1.0"/>
+        <limit lower="${joint_lower_limit}" upper="${joint_upper_limit}" effort="${joint_effort}" velocity="${joint_velocity}"/>
     </joint>
     <link name="pan_link">
@@ -120,5 +120,5 @@
                 izz="1.0" />
         </inertial>
-	</link>
+    </link>
     <!-- Leg macro -->
     <xacro:macro name="leg" params="side position x y angle axis">
@@ -130,13 +130,13 @@
         </joint>
         <link name="leg_center_${side}${position}">
-			<inertial>
-				<origin xyz="0.0 0.0 0.0" rpy="0.0 0.0 0.0" />
-				<mass value="0.00001"/>
-				<inertia
-					ixx="1.0" ixy="0.0"  ixz="0.0"
-					iyy="1.0" iyz="0.0"
-					izz="1.0" />
-			</inertial>
-		</link>
+            <inertial>
+                <origin xyz="0.0 0.0 0.0" rpy="0.0 0.0 0.0" />
+                <mass value="0.00001"/>
+                <inertia
+                    ixx="1.0" ixy="0.0"  ixz="0.0"
+                    iyy="1.0" iyz="0.0"
+                    izz="1.0" />
+            </inertial>
+        </link>
         <!-- coxa -->
         <joint name="coxa_joint_${side}${position}" type="revolute">
@@ -339,14 +339,14 @@
         </joint>
         <link name="foot_${side}${position}">
-	        <inertial>
-				<origin xyz="0.0 0.0 0.0" rpy="0.0 0.0 0.0" />
-                <mass value="0.00001"/>
-                <inertia
-                    ixx="1.0" ixy="0.0"  ixz="0.0"
-                    iyy="1.0" iyz="0.0"
-                    izz="1.0" />
-            </inertial>
-		</link>
-		<gazebo>
+            <inertial>
+                <origin xyz="0.0 0.0 0.0" rpy="0.0 0.0 0.0" />
+                <mass value="0.00001"/>
+                <inertia
+                    ixx="1.0" ixy="0.0"  ixz="0.0"
+                    iyy="1.0" iyz="0.0"
+                    izz="1.0" />
+            </inertial>
+        </link>
+        <gazebo>
             <plugin name="f3d_controller" filename="libgazebo_ros_f3d.so">
                 <alwaysOn>true</alwaysOn>
