Commit message: rework of calculated odometry into locomotion node due to latency issues

File: hexapod_description/urdf/hexapod_model.xacro (robot description, xacro)
@@ -86,5 +86,5 @@
         <parent link="base_link"/>
         <child link="imu_link"/>
-        <origin xyz="0.0 0.0 0.034" rpy="${pi} 0.0 0.0"/>
+        <origin xyz="0.0 0.0 0.034" rpy="0.0 0.0 0.0"/>
     </joint>
     <link name="imu_link">

Commit message: rework of calculated odometry into locomotion node due to latency issues

File: hexapod_description/urdf/hexapod_model.xacro (robot description, xacro)
@@ -18,5 +18,5 @@
         <parent link="base_link"/>
         <child link="body_link"/>
-        <origin xyz="0.0 0.0 0.0" rpy="0.0 0.0 0.0"/>
+        <origin xyz="0.0 0.0 0.064" rpy="0.0 0.0 0.0"/>
     </joint>
     <link name="body_link">
@@ -84,5 +84,5 @@
     <!-- IMU properties -->
     <joint name="imu_joint" type="fixed">
-        <parent link="base_link"/>
+        <parent link="body_link"/>
         <child link="imu_link"/>
         <origin xyz="0.0 0.0 0.034" rpy="0.0 0.0 0.0"/>
